Commit message: gripper

File: robot/rm_65.urdf (robot description, URDF)
Before this commit: robot rm_65_description, 7 links, 6 joints
Links:
- added link 4C2_Link1, mass 0.0024292; collision mesh filename=./meshes/4C2_Link1.STL; visual mesh filename=./meshes/4C2_Link1.STL
- added link 4C2_Link2, mass 0.0038971; collision mesh filename=./meshes/4C2_Link2.STL; visual mesh filename=./meshes/4C2_Link2.STL
- added link 4C2_Link3, mass 0.0038971; collision mesh filename=./meshes/4C2_Link3.STL; visual mesh filename=./meshes/4C2_Link3.STL
- added link 4C2_Link4, mass 0.0024292; collision mesh filename=./meshes/4C2_Link4.STL; visual mesh filename=./meshes/4C2_Link4.STL
- added link 4C2_Link5, mass 0.0045068; collision mesh filename=./meshes/4C2_Link5.STL; visual mesh filename=./meshes/4C2_Link5.STL
- added link 4C2_Link6, mass 0.0045068; collision mesh filename=./meshes/4C2_Link6.STL; visual mesh filename=./meshes/4C2_Link6.STL
- added link 4C2_baselink, mass 0.072633; collision mesh filename=./meshes/4C2_baselink.STL; visual mesh filename=./meshes/4C2_baselink.STL
Joints:
- added joint 4C2_Joint1: type revolute, parent 4C2_baselink, child 4C2_Link1, origin xyz=-0.04 -0.009 0.079 rpy=0 0 0, axis 0 -1 0, limit lower=0 upper=0.82 effort=1 velocity=1
- added joint 4C2_Joint2: type revolute, parent 4C2_baselink, child 4C2_Link2, origin xyz=-0.03 -0.009 0.081 rpy=0 0 0, axis 0 -1 0, limit lower=0 upper=0.82 effort=1 velocity=1, mimic joint=4C2_Joint1
- added joint 4C2_Joint3: type revolute, parent 4C2_baselink, child 4C2_Link3, origin xyz=0.03 -0.009 0.081 rpy=0 0 0, axis 0 -1 0, limit lower=-0.82 upper=0 effort=1 velocity=1, mimic joint=4C2_Joint1 multiplier=-1 offset=0
- added joint 4C2_Joint4: type revolute, parent 4C2_baselink, child 4C2_Link4, origin xyz=0.04 -0.009 0.079 rpy=0 0 0, axis 0 -1 0, limit lower=-0.82 upper=0 effort=1 velocity=1, mimic joint=4C2_Joint1 multiplier=-1 offset=0
- added joint 4C2_Joint5: type revolute, parent 4C2_Link1, child 4C2_Link5, origin xyz=0.0223 0.003 0.035591 rpy=0 0 0, axis 0 1 0, limit lower=0 upper=0.82 effort=1 velocity=1, mimic joint=4C2_Joint1
- added joint 4C2_Joint6: type revolute, parent 4C2_Link4, child 4C2_Link6, origin xyz=-0.0223 0.003 0.035591 rpy=0 0 0, axis 0 -1 0, limit lower=0 upper=0.82 effort=1 velocity=1, mimic joint=4C2_Joint1
- added joint sensor_joint: type fixed, parent Link6, child 4C2_baselink, origin xyz=0 0 0 rpy=0 0 1.571
