Commit message: grab animation

File: robot/arm.urdf (robot description, URDF)
Before this commit: robot rm_65_description, 14 links, 13 joints
Links:
- removed link 4C2_Link1
- removed link 4C2_Link2
- removed link 4C2_Link3
- removed link 4C2_Link4
- removed link 4C2_Link5
- removed link 4C2_Link6
- removed link 4C2_baselink
Joints:
- removed joint 4C2_Joint1
- removed joint 4C2_Joint2
- removed joint 4C2_Joint3
- removed joint 4C2_Joint4
- removed joint 4C2_Joint5
- removed joint 4C2_Joint6
- removed joint sensor_joint
- joint joint6: origin xyz=0 -0.144 0 rpy=1.5708 0 0 -> xyz=0 -0.28 0 rpy=1.5708 0 0
